Commit message: add wheel, fix tm_arm moveit bug, and add figures

File: src/mars_lite_description/urdf/mars_lite_with_gripper.urdf.xacro (robot description, xacro)
@@ -43,15 +43,13 @@
     </visual>
     <collision>
-      <!-- <origin rpy="0 0 0" xyz="${mob_base_length/2-mob_base_lower_plate_length/2} 0 ${mob_base_height/2}"/> -->
       <origin xyz="0 0 ${mob_base_height/2 - wheel_radius * 0.5}" rpy="0 0 0"/>
       <geometry>
-        <box size="${mob_base_lower_plate_length} ${mob_base_width} ${mob_base_height + wheel_radius * 0.5}"/>
+        <box size="${mob_base_lower_plate_length} ${mob_base_width} ${mob_base_height + wheel_radius * 1.0}"/>
       </geometry>
     </collision>
     <inertial>
-      <!-- <origin xyz="${mob_base_length/2-mob_base_lower_plate_length/2} 0 ${mob_base_height/2}" rpy="0 0 0" /> -->
       <origin xyz="0 0 ${mob_base_height/2 - wheel_radius * 0.5}" rpy="0 0 0" />
       <mass value="160.0" />
-      <box_inertia m="160.0" x="${mob_base_lower_plate_length}" y="${mob_base_width}" z="${mob_base_height + wheel_radius * 0.5}" />
+      <box_inertia m="160.0" x="${mob_base_lower_plate_length}" y="${mob_base_width}" z="${mob_base_height + wheel_radius * 1.0}" />
     </inertial>
   </link>
@@ -71,5 +69,4 @@
         </geometry>
       </collision>
-      <!-- <xacro:default_inertial mass="1"/> -->
       <inertial>
         <origin xyz="0 0 0" rpy="0 0 0" />
@@ -83,22 +80,18 @@
       <child link="${prefix}_wheel"/>
       <origin xyz="0 ${reflect*wheels_distance/2} 0" rpy="0 0 0"/>
-      <!-- <joint_properties damping="1.0" friction="0.0"/> -->
-      <!-- <limit effort="10000" velocity="10000"/> -->
     </joint>
   </xacro:macro>
-  <!-- <xacro:wheel prefix="right" reflect="-1"/> -->
-  <!-- <xacro:wheel prefix="left" reflect="1"/> -->
-  <!-- tm common stuff -->
+  <xacro:wheel prefix="right" reflect="-1"/>
+  <xacro:wheel prefix="left" reflect="1"/>
+  <!-- tm5 gazebo common stuff -->
   <xacro:include filename="$(find tm5_description)/urdf/common.gazebo.xacro" />
   <!-- tm5_700 -->
   <xacro:include filename="$(find tm5_description)/urdf/tm5_700.urdf.xacro" />
   <!-- arm instance -->
-  <xacro:tm5_700_robot prefix="tm_" joint_limited="false" stl_mesh="true" />
+  <xacro:tm5_700_robot prefix="tm_" joint_limited="true" stl_mesh="true" />
   <joint name="base_link_to_tm_base_link" type="fixed">
     <parent link="base_link" />
     <child link = "tm_base" />
     <origin xyz="${tm_x_offset} 0.0 ${mob_base_height}" rpy="0.0 0.0 0.0" />
-    <joint_properties damping="1000.0" friction="10000.0"/>
-    <limit effort="10000" velocity="10000"/>
   </joint>
   <!-- Frame for gripper TCP  -->

File: src/tmr_ros1_simplified_edition/tm5_description/urdf/common.gazebo.xacro (robot description, xacro)
@@ -3,6 +3,6 @@
   <gazebo>
     <plugin name="ros_control" filename="libgazebo_ros_control.so">
-      <!--robotNamespace>/</robotNamespace-->
-      <!--robotSimType>gazebo_ros_control/DefaultRobotHWSim</robotSimType-->
+      <!-- <robotNamespace>/</robotNamespace> -->
+      <!-- <robotSimType>gazebo_ros_control/DefaultRobotHWSim</robotSimType> -->
     </plugin>
 <!--

Commit message: add robotiq_85_gripper

File: src/mars_lite_description/urdf/mars_lite_with_gripper.urdf.xacro (robot description, xacro)
@@ -107,3 +107,7 @@
     <origin xyz="0 0 0" rpy="0 0 1.5708" />
   </xacro:robotiq_2f_85>   -->
+  <xacro:include filename="$(find robotiq_description)/urdf/robotiq_85_gripper.urdf.xacro" />
+  <xacro:robotiq_85_gripper prefix="" parent="tm_flange_link" >
+    <origin xyz="0 0 0" rpy="${-pi / 2} ${-pi / 2} 0"/>
+  </xacro:robotiq_85_gripper>
 </robot>

Commit message: fix self-collision problem

File: src/mars_lite_description/urdf/mars_lite_with_gripper.urdf.xacro (robot description, xacro)
@@ -14,4 +14,9 @@
   <xacro:property name="base_to_wheels_axel" value="0.01045"/>
   <xacro:property name="mob_base_lower_plate_length" value="0.630"/>
+  <!-- TM5 robot arm contrl box properties -->
+  <xacro:property name="tm_cntrl_box_length" value="0.29"/>
+  <xacro:property name="tm_cntrl_box_width" value="0.43"/>
+  <xacro:property name="tm_cntrl_box_height" value="0.23"/>
+  <xacro:property name="tm_cntrl_box_x_offset" value="-0.125"/>
   <!-- arm positioning -->
   <xacro:property name="tm_x_offset" value="0.350"/>
@@ -50,6 +55,6 @@
     <inertial>
       <origin xyz="0 0 ${mob_base_height/2 - wheel_radius * 0.5}" rpy="0 0 0" />
-      <mass value="160.0" />
-      <box_inertia m="160.0" x="${mob_base_lower_plate_length}" y="${mob_base_width}" z="${mob_base_height + wheel_radius * 1.0}" />
+      <mass value="80.0" />
+      <box_inertia m="80.0" x="${mob_base_lower_plate_length}" y="${mob_base_width}" z="${mob_base_height + wheel_radius * 1.0}" />
     </inertial>
   </link>
@@ -84,9 +89,28 @@
   <xacro:wheel prefix="right" reflect="-1"/>
   <xacro:wheel prefix="left" reflect="1"/>
-  <!-- tm5 gazebo common stuff -->
+  <!-- Robot arm contrl box -->
+  <link name="tm_cntrl_box">
+    <collision>
+      <origin xyz="0 0 0" rpy="0 0 0"/>
+      <geometry>
+        <box size="${tm_cntrl_box_length} ${tm_cntrl_box_width} ${tm_cntrl_box_height}"/>
+      </geometry>
+    </collision>
+    <inertial>
+      <origin xyz="0 0 0" rpy="0 0 0"/>
+      <mass value="5.0" />
+      <box_inertia m="5.0" x="${tm_cntrl_box_length}" y="${tm_cntrl_box_width}" z="${tm_cntrl_box_height}" />
+    </inertial>
+  </link>
+  <joint name="base_link_to_cntrl_box" type="fixed">
+      <axis xyz="0 0 0" rpy="0 0 0" />
+      <parent link="base_link"/>
+      <child link="tm_cntrl_box"/>
+      <origin xyz="${tm_cntrl_box_x_offset} 0 ${mob_base_height + tm_cntrl_box_height/2}" rpy="0 0 0"/>
+  </joint>
+  <!-- tm5_700 gazebo common stuff -->
   <xacro:include filename="$(find tm5_description)/urdf/common.gazebo.xacro" />
   <!-- tm5_700 -->
   <xacro:include filename="$(find tm5_description)/urdf/tm5_700.urdf.xacro" />
-  <!-- arm instance -->
   <xacro:tm5_700_robot prefix="tm_" joint_limited="true" stl_mesh="true" />
   <joint name="base_link_to_tm_base_link" type="fixed">
@@ -95,16 +119,5 @@
     <origin xyz="${tm_x_offset} 0.0 ${mob_base_height}" rpy="0.0 0.0 0.0" />
   </joint>
-  <!-- Frame for gripper TCP  -->
-  <!-- <link name="tm_gripper"/>
-  <joint name="tm_tip_link_to_tm_gripper" type="fixed">
-    <parent link="tm_tip_link"/>
-    <child link="tm_gripper"/>
-    <origin xyz="0 0 ${0.1628+0.0139}" rpy="0 0 0"/>
-  </joint> -->
-  <!-- Robotiq from Beta Robots fork-->
-  <!-- <xacro:include filename="$(find robotiq_2f_model)/model/robotiq_2f_85.urdf.xacro" />
-  <xacro:robotiq_2f_85 name="gripper" parent="tm_tip_link" precise_collision="false" adaptive_transmission="false">
-    <origin xyz="0 0 0" rpy="0 0 1.5708" />
-  </xacro:robotiq_2f_85>   -->
+  <!-- Robotiq 85 gripper -->
   <xacro:include filename="$(find robotiq_description)/urdf/robotiq_85_gripper.urdf.xacro" />
   <xacro:robotiq_85_gripper prefix="" parent="tm_flange_link" >

Commit message: fix noetic incompatible setup

File: src/mars_lite_description/urdf/mars_lite_with_gripper.urdf.xacro (robot description, xacro)
@@ -56,7 +56,14 @@
       <origin xyz="0 0 ${mob_base_height/2 - wheel_radius * 0.5}" rpy="0 0 0" />
       <mass value="80.0" />
-      <box_inertia m="80.0" x="${mob_base_lower_plate_length}" y="${mob_base_width}" z="${mob_base_height + wheel_radius * 1.0}" />
+      <xacro:box_inertia m="80.0" x="${mob_base_lower_plate_length}" y="${mob_base_width}" z="${mob_base_height + wheel_radius * 1.0}" />
     </inertial>
   </link>
+  <!-- Dummy footprint link -->
+  <!-- <link name="base_footprint" />
+  <joint name="footprint_joint" type="fixed">
+      <origin xyz="0 0 0" rpy="0 0 0" />
+      <parent link="base_footprint"/>
+      <child link="base_link"/>
+  </joint> -->
   <!-- Wheels -->
   <xacro:macro name="wheel" params="prefix reflect">
@@ -77,5 +84,5 @@
         <origin xyz="0 0 0" rpy="0 0 0" />
         <mass value="10" />
-        <cylinder_inertia m="10" r="${wheel_radius}" h="0.03" />
+        <xacro:cylinder_inertia m="10" r="${wheel_radius}" h="0.03" />
       </inertial>
     </link>
@@ -100,5 +107,5 @@
       <origin xyz="0 0 0" rpy="0 0 0"/>
       <mass value="5.0" />
-      <box_inertia m="5.0" x="${tm_cntrl_box_length}" y="${tm_cntrl_box_width}" z="${tm_cntrl_box_height}" />
+      <xacro:box_inertia m="5.0" x="${tm_cntrl_box_length}" y="${tm_cntrl_box_width}" z="${tm_cntrl_box_height}" />
     </inertial>
   </link>

Commit message: fix noetic incompatible setup

File: src/mars_lite_description/urdf/mars_lite_with_gripper.urdf.xacro (robot description, xacro)
@@ -42,5 +42,5 @@
   <link name="base_link">
     <visual>
-      <origin rpy="0 0 0" xyz="0 0 0"/>
+      <origin xyz="0 0 0" rpy="0 0 0"/>
       <geometry>
           <mesh filename="package://mars_lite_description/meshes/mob_plat.dae"/>
@@ -62,7 +62,7 @@
   <!-- <link name="base_footprint" />
   <joint name="footprint_joint" type="fixed">
-      <origin xyz="0 0 0" rpy="0 0 0" />
-      <parent link="base_footprint"/>
-      <child link="base_link"/>
+      <origin xyz="0 0 ${-wheel_radius * 0.5}" rpy="0 0 0" />
+      <parent link="base_link"/>
+      <child link="base_footprint"/>
   </joint> -->
   <!-- Wheels -->

Commit message: fix ros noetic version bug

File: src/mars_lite_description/urdf/mars_lite_with_gripper.urdf.xacro (robot description, xacro)
@@ -87,5 +87,5 @@
       </inertial>
     </link>
-    <joint name="${prefix}_wheel" type="continuous">
+    <joint name="${prefix}_wheel_joint" type="continuous">
       <axis xyz="0 1 0" rpy="0 0 0" />
       <parent link="base_link"/>

Commit message: add laser and realsense

File: src/mars_lite_description/urdf/mars_lite_with_gripper.urdf.xacro (robot description, xacro)
@@ -1,5 +1,7 @@
 <?xml version="1.0"?>
-<robot name="mars_lite"
-  xmlns:xacro="http://www.ros.org/wiki/xacro">
+<robot name="mars_lite" xmlns:xacro="http://www.ros.org/wiki/xacro">
+  <!-- Arguments -->
+  <xacro:arg name="laser_enabled" default="1" />
+  <xacro:arg name="realsense_enabled" default="0" />
   <!-- Gazebo plugin -->
   <xacro:include filename="$(find mars_lite_description)/urdf/mars_lite.gazebo" />
@@ -48,23 +50,55 @@
     </visual>
     <collision>
-      <origin xyz="0 0 ${mob_base_height/2 - wheel_radius * 0.5}" rpy="0 0 0"/>
+      <origin xyz="0 0 ${mob_base_height / 2 + 0.05}" rpy="0 0 0"/>
       <geometry>
-        <box size="${mob_base_lower_plate_length} ${mob_base_width} ${mob_base_height + wheel_radius * 1.0}"/>
+        <box size="${mob_base_lower_plate_length} ${mob_base_width} ${mob_base_height - 0.08}"/>
       </geometry>
     </collision>
     <inertial>
-      <origin xyz="0 0 ${mob_base_height/2 - wheel_radius * 0.5}" rpy="0 0 0" />
+      <origin xyz="0 0 ${mob_base_height / 2 + 0.05}" rpy="0 0 0" />
       <mass value="80.0" />
-      <xacro:box_inertia m="80.0" x="${mob_base_lower_plate_length}" y="${mob_base_width}" z="${mob_base_height + wheel_radius * 1.0}" />
+      <xacro:box_inertia m="80.0" x="${mob_base_lower_plate_length}" y="${mob_base_width}" z="${mob_base_height - 0.08}" />
     </inertial>
   </link>
   <!-- Dummy footprint link -->
-  <!-- <link name="base_footprint" />
+  <link name="base_footprint" />
   <joint name="footprint_joint" type="fixed">
-      <origin xyz="0 0 ${-wheel_radius * 0.5}" rpy="0 0 0" />
+    <origin xyz="0 0 ${-wheel_radius}" rpy="0 0 0" />
+    <parent link="base_link"/>
+    <child link="base_footprint"/>
+  </joint>
+  <!-- Caster support -->
+  <xacro:macro name="caster_support" params="prefix reflect_fr reflect_lr">
+    <link name="${prefix}_caster_support">
+      <collision>
+          <origin xyz="0 0 ${-wheel_radius * 2}" rpy="0 0 0" />
+          <geometry>
+            <cylinder radius="0.025" length="${wheel_radius * 2}"/>
+          </geometry>
+        </collision>
+      <inertial>
+        <origin xyz="0 0 ${-wheel_radius * 2}" rpy="0 0 0" />
+        <mass value="1.0" />
+        <xacro:cylinder_inertia m="1.0" r="0.025" h="${wheel_radius * 2}" />
+      </inertial>
+    </link>
+    <joint name="${prefix}_caster_support_joint" type="fixed">
+      <origin xyz="${0.225 * reflect_fr} ${0.17 * reflect_lr} ${wheel_radius * 2}" rpy="0 0 0" />
       <parent link="base_link"/>
-      <child link="base_footprint"/>
-  </joint> -->
-  <!-- Wheels -->
+      <child link="${prefix}_caster_support"/>
+    </joint>
+    <gazebo reference="${prefix}_caster_support">
+        <mu1 value="0.01"/>
+        <mu2 value="0.01"/>
+        <kp  value="1000000.0" />
+        <kd  value="10000.0" />
+        <fdir1 value="1 0 0" />
+    </gazebo>
+  </xacro:macro>
+  <xacro:caster_support prefix="front_left" reflect_fr="1" reflect_lr="1"/>
+  <xacro:caster_support prefix="front_right" reflect_fr="1" reflect_lr="-1"/>
+  <xacro:caster_support prefix="back_left" reflect_fr="-1" reflect_lr="1"/>
+  <xacro:caster_support prefix="back_right" reflect_fr="-1" reflect_lr="-1"/>
+  <!-- Driving wheels -->
   <xacro:macro name="wheel" params="prefix reflect">
     <link name="${prefix}_wheel">
@@ -111,8 +145,8 @@
   </link>
   <joint name="base_link_to_cntrl_box" type="fixed">
-      <axis xyz="0 0 0" rpy="0 0 0" />
-      <parent link="base_link"/>
-      <child link="tm_cntrl_box"/>
-      <origin xyz="${tm_cntrl_box_x_offset} 0 ${mob_base_height + tm_cntrl_box_height/2}" rpy="0 0 0"/>
+    <axis xyz="0 0 0" rpy="0 0 0" />
+    <parent link="base_link"/>
+    <child link="tm_cntrl_box"/>
+    <origin xyz="${tm_cntrl_box_x_offset} 0 ${mob_base_height + tm_cntrl_box_height/2}" rpy="0 0 0"/>
   </joint>
   <!-- tm5_700 gazebo common stuff -->
@@ -121,9 +155,51 @@
   <xacro:include filename="$(find tm5_description)/urdf/tm5_700.urdf.xacro" />
   <xacro:tm5_700_robot prefix="tm_" joint_limited="true" stl_mesh="true" />
-  <joint name="base_link_to_tm_base_link" type="fixed">
+  <joint name="base_link_to_tm_base" type="fixed">
     <parent link="base_link" />
-    <child link = "tm_base" />
+    <child link="tm_base" />
     <origin xyz="${tm_x_offset} 0.0 ${mob_base_height}" rpy="0.0 0.0 0.0" />
   </joint>
+  <!-- Hokuyo utm30lx laser scanner -->
+  <xacro:if value="$(arg laser_enabled)">
+    <!-- Dummy merged laser frame -->
+    <link name="merged_laser_frame" />
+    <joint name="base_link_to_merged_laser_frame" type="fixed">
+      <parent link="base_link" />
+      <child link="merged_laser_frame" />
+      <origin xyz="0 0 0" rpy="0 0 0" />
+    </joint>
+    <xacro:include filename="$(find hector_sensors_description)/urdf/hokuyo_utm30lx.urdf.xacro" />
+    <!-- back_laser -->
+    <xacro:hokuyo_utm30lx name="back_laser"
+                          parent="base_link"
+                          ros_topic="back_scan"
+                          update_rate="40"
+                          ray_count="1081"
+                          min_angle="-90"
+                          max_angle="90">
+      <origin xyz="-0.285 0.00 0.05" rpy="${pi} 0 ${pi}" />
+    </xacro:hokuyo_utm30lx>
+    <!-- front_laser -->
+    <xacro:hokuyo_utm30lx name="front_laser"
+                          parent="base_link"
+                          ros_topic="front_scan"
+                          update_rate="40"
+                          ray_count="1081"
+                          min_angle="-90"
+                          max_angle="90">
+      <origin xyz="0.285 0.00 0.05" rpy="${-pi} 0 0" />
+    </xacro:hokuyo_utm30lx>
+  </xacro:if>
+  <!-- Intel realsense D435 -->
+  <xacro:if value="$(arg realsense_enabled)">
+  <xacro:include filename="$(find mars_lite_description)/urdf/accessories/intel_realsense.urdf.xacro"/>
+    <xacro:intel_realsense_mount prefix="camera1" topic="camera1" parent_link="realsense_mount"/>
+    <link name="realsense_mount"/>
+    <joint name="realsense_mount_joint" type="fixed">
+      <origin xyz="0 0.05 0.062" rpy="0 ${-pi / 2} ${-pi / 2}" />
+      <parent link="tm_wrist_3_link"/>
+      <child link="realsense_mount" />
+    </joint>
+  </xacro:if>
   <!-- Robotiq 85 gripper -->
   <xacro:include filename="$(find robotiq_description)/urdf/robotiq_85_gripper.urdf.xacro" />
